Commit message: siiim

File: buffpy/config/robots/infantry-sim/buffbot.xacro (robot description, xacro)
@@ -39,66 +39,63 @@
       </link>
   </xacro:macro>
-  <xacro:macro name="default_box_link" params="link_name x y z color mass">
+  <xacro:macro name="no_collision_cylinder_link" params="link_name radius length color mass">
     <link name="${link_name}">
         <visual>
          <origin xyz="0 0 0" rpy="0 0 0" />
          <geometry>
-           <box size="${x} ${y} ${z}"/>
+           <cylinder radius="${radius}" length="${length}"/>
          </geometry>
          <material name="${color}"/>
        </visual>
-       <collision>
-         <origin xyz="0 0 0" rpy="0 0 0" />
-         <geometry>
-           <box size="${x} ${y} ${z}"/>
-         </geometry>
-       </collision>
        <inertial>
          <origin xyz="0 0 0" rpy="0 0 0"/>
          <mass value="${mass}"/>
-         <inertia ixx="${(1/12) * ((z * z) + (y * y)) * mass}"  ixy="0"  ixz="0"
-          iyy="${(1/12) * ((x * x) + (z * z)) * mass}" iyz="0" izz="${(1/12) * ((x * x) + (y * y)) * mass}" />
+         <inertia ixx="${(1/12) * ((length * length) + (3 * (radius * radius))) * mass}"  ixy="0"  ixz="0"
+          iyy="${(1/12) * ((length * length) + (3 * (radius * radius))) * mass}" iyz="0" izz="${(1/2) * mass * radius * radius}" />
        </inertial>
       </link>
   </xacro:macro>
-  <xacro:macro name="swerve" params="id w l g">
-    <xacro:default_cylinder_link link_name="${id}_swerve" radius="${w*0.25}" length="0.05" color="black" mass="25"/>
+  <xacro:macro name="default_box_link" params="link_name x y z color mass">
+    <link name="${link_name}">
+      <visual>
+        <origin xyz="0 0 0" rpy="0 0 0" />
+        <geometry>
+          <box size="${x} ${y} ${z}"/>
+        </geometry>
+       <material name="${color}"/>
+      </visual>
+      <collision>
+        <origin xyz="0 0 0" rpy="0 0 0" />
+        <geometry>
+          <box size="${x} ${y} ${z}"/>
+        </geometry>
+      </collision>
+      <inertial>
+        <origin xyz="0 0 0" rpy="0 0 0"/>
+        <mass value="${mass}"/>
+        <inertia ixx="${(1/12) * ((z * z) + (y * y)) * mass}"  ixy="0"  ixz="0"
+          iyy="${(1/12) * ((x * x) + (z * z)) * mass}" iyz="0" izz="${(1/12) * ((x * x) + (y * y)) * mass}" />
+      </inertial>
+    </link>
+  </xacro:macro>
+  <xacro:macro name="swerve_hub" params="id l w x y">
+    <xacro:default_cylinder_link link_name="${id}_swerve" radius="${w*0.3}" length="0.06" color="black" mass="5"/>
     <gazebo reference="${id}_swerve">
       <material>Gazebo/Black</material>
-      <selfCollide>True</selfCollide>
+      <selfCollide>true</selfCollide>
+      <static>false</static>
     </gazebo>
     <joint name="${id}_steer" type="continuous">
       <parent link="base_link"/>
       <child link="${id}_swerve"/>
-      <origin xyz="${l} ${w} ${g - 0.025}"/>
+      <origin xyz="${x * l} ${y * w} 0"/>
       <axis xyz="0 0 1"/>
     </joint>
-    <transmission name="tran_s_${id}">
+    <transmission name="trans_${id}">
       <type>transmission_interface/SimpleTransmission</type>
       <joint name="${id}_steer">
         <hardwareInterface>hardware_interface/EffortJointInterface</hardwareInterface>
       </joint>
-      <actuator name="${id}_steer">
-        <hardwareInterface>hardware_interface/EffortJointInterface</hardwareInterface>
-        <mechanicalReduction>1</mechanicalReduction>
-      </actuator>
-    </transmission>
-    <xacro:default_cylinder_link link_name="${id}_wheel" radius="${w*0.15}" length="0.025" color="light-gray" mass="50"/>
-    <gazebo reference="${id}_wheel">
-      <material>Gazebo/White</material>
-      <selfCollide>True</selfCollide>
-    </gazebo>
-    <joint name="${id}_drive" type="continuous">
-      <parent link="${id}_swerve"/>
-      <child link="${id}_wheel"/>
-      <origin xyz="0 0 ${g - 0.075}" rpy="1.57 0 0"/>
-      <axis xyz="0 0 1"/>
-    </joint>
-    <transmission name="tran_d_${id}">
-      <type>transmission_interface/SimpleTransmission</type>
-      <joint name="${id}_drive">
-        <hardwareInterface>hardware_interface/EffortJointInterface</hardwareInterface>
-      </joint>
-      <actuator name="${id}_drive">
+      <actuator name="${id}_steer_motor">
         <hardwareInterface>hardware_interface/EffortJointInterface</hardwareInterface>
         <mechanicalReduction>1</mechanicalReduction>
@@ -106,27 +103,66 @@
     </transmission>
   </xacro:macro>
+  <xacro:macro name="swerve_indicator" params="l w x y">
+    <xacro:no_collision_cylinder_link link_name="swerve_ind" radius="${w*0.26}" length="0.075" color="gold" mass="0"/>
+    <gazebo reference="swerve_ind">
+      <material>Gazebo/Gold</material>
+      <selfCollide>true</selfCollide>
+      <static>false</static>
+    </gazebo>
+    <joint name="swerve_xy" type="fixed">
+      <parent link="base_link"/>
+      <child link="swerve_ind"/>
+      <origin xyz="${x * l} ${y * w} 0"/>
+      <axis xyz="0 0 1"/>
+    </joint>
+  </xacro:macro>
+  <xacro:macro name="swerve_wheel" params="id l w x y">
+    <xacro:default_cylinder_link link_name="${id}_wheel" radius="${w*0.15}" length="0.025" color="light-gray" mass="5"/>
+    <gazebo reference="${id}_wheel">
+      <material>Gazebo/White</material>
+      <selfCollide>true</selfCollide>
+      <static>false</static>
+      <kp>1000000.0</kp>
+      <kd>100.0</kd>
+      <mu1>1.0</mu1>
+      <mu2>1.0</mu2>
+    </gazebo>
+    <joint name="${id}_drive" type="continuous">
+      <parent link="${id}_swerve"/>
+      <child link="${id}_wheel"/>
+      <origin xyz="0 0 ${w*-0.16}" rpy="1.57 0 0"/>
+      <axis xyz="0 0 1"/>
+    </joint>
+    <transmission name="trand_${id}">
+      <type>transmission_interface/SimpleTransmission</type>
+      <joint name="${id}_drive">
+        <hardwareInterface>hardware_interface/EffortJointInterface</hardwareInterface>
+      </joint>
+      <actuator name="${id}_drive_motor">
+        <hardwareInterface>hardware_interface/EffortJointInterface</hardwareInterface>
+        <mechanicalReduction>1</mechanicalReduction>
+      </actuator>
+    </transmission>
+  </xacro:macro>
+  <xacro:macro name="swerve" params="id l w x y">
+    <xacro:swerve_hub id="${id}" l="${l}" w="${w}" x="${x}" y="${y}"/>
+    <xacro:swerve_wheel id="${id}" l="${l}" w="${w}" x="${x}" y="${y}"/>
+  </xacro:macro>
   <xacro:macro name="swerve_chassis" params="w l g">
-    <xacro:default_box_link link_name="base_link" x="${l * 2}" y="${w * 2}" z="${0.025}" color="black" mass="20"/>
+    <xacro:default_box_link link_name="base_link" x="${l * 2}" y="${w * 2}" z="${0.025}" color="black" mass="10"/>
     <gazebo reference="base_link">
       <material>Gazebo/Black</material>
-      <selfCollide>True</selfCollide>
+      <selfCollide>true</selfCollide>
+      <static>false</static>
+      <mu1>0.5</mu1>
+      <mu2>0.5</mu2>
     </gazebo>
-    <xacro:swerve id="fl" w="${w}" l="${l}" g="${g}"/>
-    <xacro:swerve id="fr" w="-${w}" l="${l}" g="${g}"/>
-    <xacro:swerve id="rr" w="-${w}" l="-${l}" g="${g}"/>
-    <xacro:swerve id="rl" w="${w}" l="-${l}" g="${g}"/>
-    <xacro:default_cylinder_link link_name="fl_swerve_mark" radius="${w*0.2}" length="0.051" color="black" mass="0.1"/>
-    <joint name="fl_swerve_marker" type="fixed">
-      <parent link="base_link"/>
-      <child link="fl_swerve_mark"/>
-      <origin xyz="${l} ${w} ${g - 0.025}"/>
-      <axis xyz="0 0 1"/>
-    </joint>
-    <gazebo reference="fl_swerve_mark">
-      <material>Gazebo/Gold</material>
-      <selfCollide>True</selfCollide>
-    </gazebo>
+    <xacro:swerve id="fl" l="${l}" w="${w}" x="1" y="1"/>
+    <xacro:swerve id="fr" l="${l}" w="${w}" x="-1" y="1"/>
+    <xacro:swerve id="rr" l="${l}" w="${w}" x="-1" y="-1"/>
+    <xacro:swerve id="rl" l="${l}" w="${w}" x="1" y="-1"/>
+    <xacro:swerve_indicator l="${l}" w="${w}" x="1" y="1"/>
   </xacro:macro>
-  <xacro:swerve_chassis w="0.17" l="0.17" g="0.045"/>
+  <xacro:swerve_chassis w="0.17" l="0.17" g="0.1"/>
   <gazebo>
     <plugin name="gazebo_ros_control" filename="libgazebo_ros_control.so">

File: buffpy/config/robots/infantry/buffbot.xacro (robot description, xacro)
@@ -16,74 +16,157 @@
     <color rgba="0.81 0.72 0.48 1"/>
   </material>
-  <xacro:macro name="swerve" params="id w l g">
-      <link name="${id}_swerve">
+  <xacro:macro name="default_cylinder_link" params="link_name radius length color mass">
+    <link name="${link_name}">
         <visual>
          <origin xyz="0 0 0" rpy="0 0 0" />
          <geometry>
-           <cylinder radius="${w*0.25}" length="0.05"/>
+           <cylinder radius="${radius}" length="${length}"/>
          </geometry>
-         <material name="black"/>
+         <material name="${color}"/>
        </visual>
        <collision>
          <origin xyz="0 0 0" rpy="0 0 0" />
          <geometry>
-           <cylinder radius="${w*0.25}" length="0.05"/>
+           <cylinder radius="${radius}" length="${length}"/>
          </geometry>
        </collision>
+       <inertial>
+         <origin xyz="0 0 0" rpy="0 0 0"/>
+         <mass value="${mass}"/>
+         <inertia ixx="${(1/12) * ((length * length) + (3 * (radius * radius))) * mass}"  ixy="0"  ixz="0"
+          iyy="${(1/12) * ((length * length) + (3 * (radius * radius))) * mass}" iyz="0" izz="${(1/2) * mass * radius * radius}" />
+       </inertial>
       </link>
-      <joint name="base_to_${id}_swerve" type="continuous">
-        <parent link="base_link"/>
-        <child link="${id}_swerve"/>
-        <origin xyz="${l} ${w} ${g - 0.025}"/>
-        <axis xyz="0 0 1"/>
-      </joint>
-      <link name="${id}_wheel">
+  </xacro:macro>
+  <xacro:macro name="no_collision_cylinder_link" params="link_name radius length color mass">
+    <link name="${link_name}">
         <visual>
          <origin xyz="0 0 0" rpy="0 0 0" />
          <geometry>
-           <cylinder radius="${w*0.15}" length="0.025"/>
+           <cylinder radius="${radius}" length="${length}"/>
          </geometry>
-         <material name="light-gray"/>
+         <material name="${color}"/>
        </visual>
-       <collision>
-         <origin xyz="0 0 0" rpy="0 0 0" />
-         <geometry>
-           <cylinder radius="${w*0.15}" length="0.025"/>
-         </geometry>
-       </collision>
+       <inertial>
+         <origin xyz="0 0 0" rpy="0 0 0"/>
+         <mass value="${mass}"/>
+         <inertia ixx="${(1/12) * ((length * length) + (3 * (radius * radius))) * mass}"  ixy="0"  ixz="0"
+          iyy="${(1/12) * ((length * length) + (3 * (radius * radius))) * mass}" iyz="0" izz="${(1/2) * mass * radius * radius}" />
+       </inertial>
       </link>
-      <joint name="${id}_swerve_to_wheel" type="continuous">
-        <parent link="${id}_swerve"/>
-        <child link="${id}_wheel"/>
-        <origin xyz="0 0 ${g - 0.075}" rpy="1.57 0 0"/>
-        <axis xyz="0 0 1"/>
+  </xacro:macro>
+  <xacro:macro name="default_box_link" params="link_name x y z color mass">
+    <link name="${link_name}">
+      <visual>
+        <origin xyz="0 0 0" rpy="0 0 0" />
+        <geometry>
+          <box size="${x} ${y} ${z}"/>
+        </geometry>
+       <material name="${color}"/>
+      </visual>
+      <collision>
+        <origin xyz="0 0 0" rpy="0 0 0" />
+        <geometry>
+          <box size="${x} ${y} ${z}"/>
+        </geometry>
+      </collision>
+      <inertial>
+        <origin xyz="0 0 0" rpy="0 0 0"/>
+        <mass value="${mass}"/>
+        <inertia ixx="${(1/12) * ((z * z) + (y * y)) * mass}"  ixy="0"  ixz="0"
+          iyy="${(1/12) * ((x * x) + (z * z)) * mass}" iyz="0" izz="${(1/12) * ((x * x) + (y * y)) * mass}" />
+      </inertial>
+    </link>
+  </xacro:macro>
+  <xacro:macro name="swerve_hub" params="id l w x y">
+    <xacro:default_cylinder_link link_name="${id}_swerve" radius="${w*0.3}" length="0.06" color="black" mass="5"/>
+    <gazebo reference="${id}_swerve">
+      <material>Gazebo/Black</material>
+      <selfCollide>true</selfCollide>
+      <static>false</static>
+    </gazebo>
+    <joint name="${id}_steer" type="continuous">
+      <parent link="base_link"/>
+      <child link="${id}_swerve"/>
+      <origin xyz="${x * l} ${y * w} 0"/>
+      <axis xyz="0 0 1"/>
+    </joint>
+    <transmission name="trans_${id}">
+      <type>transmission_interface/SimpleTransmission</type>
+      <joint name="${id}_steer">
+        <hardwareInterface>hardware_interface/EffortJointInterface</hardwareInterface>
       </joint>
+      <actuator name="${id}_steer_motor">
+        <hardwareInterface>hardware_interface/EffortJointInterface</hardwareInterface>
+        <mechanicalReduction>1</mechanicalReduction>
+      </actuator>
+    </transmission>
+  </xacro:macro>
+  <xacro:macro name="swerve_indicator" params="l w x y">
+    <xacro:no_collision_cylinder_link link_name="swerve_ind" radius="${w*0.26}" length="0.075" color="gold" mass="0"/>
+    <gazebo reference="swerve_ind">
+      <material>Gazebo/Gold</material>
+      <selfCollide>true</selfCollide>
+      <static>false</static>
+    </gazebo>
+    <joint name="swerve_xy" type="fixed">
+      <parent link="base_link"/>
+      <child link="swerve_ind"/>
+      <origin xyz="${x * l} ${y * w} 0"/>
+      <axis xyz="0 0 1"/>
+    </joint>
+  </xacro:macro>
+  <xacro:macro name="swerve_wheel" params="id l w x y">
+    <xacro:default_cylinder_link link_name="${id}_wheel" radius="${w*0.15}" length="0.025" color="light-gray" mass="5"/>
+    <gazebo reference="${id}_wheel">
+      <material>Gazebo/White</material>
+      <selfCollide>true</selfCollide>
+      <static>false</static>
+      <kp>1000000.0</kp>
+      <kd>100.0</kd>
+      <mu1>1.0</mu1>
+      <mu2>1.0</mu2>
+    </gazebo>
+    <joint name="${id}_drive" type="continuous">
+      <parent link="${id}_swerve"/>
+      <child link="${id}_wheel"/>
+      <origin xyz="0 0 ${w*-0.16}" rpy="1.57 0 0"/>
+      <axis xyz="0 0 1"/>
+    </joint>
+    <transmission name="trand_${id}">
+      <type>transmission_interface/SimpleTransmission</type>
+      <joint name="${id}_drive">
+        <hardwareInterface>hardware_interface/EffortJointInterface</hardwareInterface>
+      </joint>
+      <actuator name="${id}_drive_motor">
+        <hardwareInterface>hardware_interface/EffortJointInterface</hardwareInterface>
+        <mechanicalReduction>1</mechanicalReduction>
+      </actuator>
+    </transmission>
+  </xacro:macro>
+  <xacro:macro name="swerve" params="id l w x y">
+    <xacro:swerve_hub id="${id}" l="${l}" w="${w}" x="${x}" y="${y}"/>
+    <xacro:swerve_wheel id="${id}" l="${l}" w="${w}" x="${x}" y="${y}"/>
   </xacro:macro>
   <xacro:macro name="swerve_chassis" params="w l g">
-    <link name="base_link">
-      <inertial>
-       <origin xyz="0 0 ${g}" rpy="0 0 0"/>
-       <mass value="1"/>
-       <inertia ixx="100"  ixy="0"  ixz="0" iyy="100" iyz="0" izz="100" />
-     </inertial>
-     <visual>
-       <origin xyz="0 0 ${g}" rpy="0 0 0" />
-       <geometry>
-         <box size="${l * 2} ${w * 2} 0.025"/>
-       </geometry>
-       <material name="black"/>
-     </visual>
-     <collision>
-       <origin xyz="0 0 0.05" rpy="0 0 0"/>
-       <geometry>
-         <box size="${l * 2} ${w * 2} 0.025"/>
-       </geometry>
-     </collision>
-    </link>
-    <xacro:swerve id="fl" w="${w}" l="${l}" g="${g}"/>
-    <xacro:swerve id="fr" w="-${w}" l="${l}" g="${g}"/>
-    <xacro:swerve id="rr" w="-${w}" l="-${l}" g="${g}"/>
-    <xacro:swerve id="rl" w="${w}" l="-${l}" g="${g}"/>
+    <xacro:default_box_link link_name="base_link" x="${l * 2}" y="${w * 2}" z="${0.025}" color="black" mass="10"/>
+    <gazebo reference="base_link">
+      <material>Gazebo/Black</material>
+      <selfCollide>true</selfCollide>
+      <static>false</static>
+      <mu1>0.5</mu1>
+      <mu2>0.5</mu2>
+    </gazebo>
+    <xacro:swerve id="fl" l="${l}" w="${w}" x="1" y="1"/>
+    <xacro:swerve id="fr" l="${l}" w="${w}" x="-1" y="1"/>
+    <xacro:swerve id="rr" l="${l}" w="${w}" x="-1" y="-1"/>
+    <xacro:swerve id="rl" l="${l}" w="${w}" x="1" y="-1"/>
+    <xacro:swerve_indicator l="${l}" w="${w}" x="1" y="1"/>
   </xacro:macro>
-  <xacro:swerve_chassis w="0.17" l="0.17" g="0.045"/>
+  <xacro:swerve_chassis w="0.17" l="0.17" g="0.1"/>
+  <gazebo>
+    <plugin name="gazebo_ros_control" filename="libgazebo_ros_control.so">
+      <robotNamespace>/buffbot</robotNamespace>
+    </plugin>
+  </gazebo>
 </robot>

Commit message: lots of stuff

File: buffpy/config/robots/infantry-sim/buffbot.xacro (robot description, xacro)
@@ -131,5 +131,5 @@
       <parent link="${id}_swerve"/>
       <child link="${id}_wheel"/>
-      <origin xyz="0 0 ${w*-0.16}" rpy="1.57 0 0"/>
+      <origin xyz="0 0 ${w*-0.16}" rpy="${pi / 2.0} 0 0"/>
       <axis xyz="0 0 1"/>
     </joint>
@@ -158,8 +158,8 @@
       <mu2>0.5</mu2>
     </gazebo>
-    <xacro:swerve id="fl" l="${l}" w="${w}" x="1" y="1" a="${3.14 / 4}"/>
-    <xacro:swerve id="fr" l="${l}" w="${w}" x="1" y="-1" a="${-3.14 / 4}"/>
-    <xacro:swerve id="rr" l="${l}" w="${w}" x="-1" y="-1" a="${-3.14 / 4 * 3}"/>
-    <xacro:swerve id="rl" l="${l}" w="${w}" x="-1" y="1" a="${3.14 / 4 * 3}"/>
+    <xacro:swerve id="fl" l="${l}" w="${w}" x="1" y="1" a="${pi / 4}"/>
+    <xacro:swerve id="fr" l="${l}" w="${w}" x="1" y="-1" a="${-pi / 4}"/>
+    <xacro:swerve id="rr" l="${l}" w="${w}" x="-1" y="-1" a="${-pi / 4 * 3}"/>
+    <xacro:swerve id="rl" l="${l}" w="${w}" x="-1" y="1" a="${pi / 4 * 3}"/>
     <xacro:swerve_indicator l="${l}" w="${w}" x="1" y="1"/>
   </xacro:macro>

File: buffpy/config/robots/infantry/buffbot.xacro (robot description, xacro)
@@ -79,5 +79,5 @@
     </link>
   </xacro:macro>
-  <xacro:macro name="swerve_hub" params="id l w x y">
+  <xacro:macro name="swerve_hub" params="id l w x y a">
     <xacro:default_cylinder_link link_name="${id}_swerve" radius="${w*0.3}" length="0.06" color="black" mass="5"/>
     <gazebo reference="${id}_swerve">
@@ -89,5 +89,5 @@
       <parent link="base_link"/>
       <child link="${id}_swerve"/>
-      <origin xyz="${x * l} ${y * w} 0"/>
+      <origin xyz="${x * l} ${y * w} 0" rpy="0 0 ${a}"/>
       <axis xyz="0 0 1"/>
     </joint>
@@ -131,5 +131,5 @@
       <parent link="${id}_swerve"/>
       <child link="${id}_wheel"/>
-      <origin xyz="0 0 ${w*-0.16}" rpy="1.57 0 0"/>
+      <origin xyz="0 0 ${w*-0.16}" rpy="${pi / 2.0} 0 0"/>
       <axis xyz="0 0 1"/>
     </joint>
@@ -145,6 +145,6 @@
     </transmission>
   </xacro:macro>
-  <xacro:macro name="swerve" params="id l w x y">
-    <xacro:swerve_hub id="${id}" l="${l}" w="${w}" x="${x}" y="${y}"/>
+  <xacro:macro name="swerve" params="id l w x y a">
+    <xacro:swerve_hub id="${id}" l="${l}" w="${w}" x="${x}" y="${y}" a="${a}"/>
     <xacro:swerve_wheel id="${id}" l="${l}" w="${w}" x="${x}" y="${y}"/>
   </xacro:macro>
@@ -158,8 +158,8 @@
       <mu2>0.5</mu2>
     </gazebo>
-    <xacro:swerve id="fl" l="${l}" w="${w}" x="1" y="1"/>
-    <xacro:swerve id="fr" l="${l}" w="${w}" x="-1" y="1"/>
-    <xacro:swerve id="rr" l="${l}" w="${w}" x="-1" y="-1"/>
-    <xacro:swerve id="rl" l="${l}" w="${w}" x="1" y="-1"/>
+    <xacro:swerve id="fl" l="${l}" w="${w}" x="1" y="1" a="${pi / 4}"/>
+    <xacro:swerve id="fr" l="${l}" w="${w}" x="1" y="-1" a="${-pi / 4}"/>
+    <xacro:swerve id="rr" l="${l}" w="${w}" x="-1" y="-1" a="${-pi / 4 * 3}"/>
+    <xacro:swerve id="rl" l="${l}" w="${w}" x="-1" y="1" a="${pi / 4 * 3}"/>
     <xacro:swerve_indicator l="${l}" w="${w}" x="1" y="1"/>
   </xacro:macro>

File: buffpy/config/robots/penguin/buffbot.xacro (robot description, xacro)
@@ -131,5 +131,5 @@
       <parent link="${id}_swerve"/>
       <child link="${id}_wheel"/>
-      <origin xyz="0 0 ${w*-0.16}" rpy="1.57 0 0"/>
+      <origin xyz="0 0 ${w*-0.16}" rpy="${pi / 2.0} 0 0"/>
       <axis xyz="0 0 1"/>
     </joint>
@@ -158,8 +158,8 @@
       <mu2>0.5</mu2>
     </gazebo>
-    <xacro:swerve id="fl" l="${l}" w="${w}" x="1" y="1" a="${3.1415926535 / 4}"/>
-    <xacro:swerve id="fr" l="${l}" w="${w}" x="1" y="-1" a="${-3.1415926535 / 4}"/>
-    <xacro:swerve id="rr" l="${l}" w="${w}" x="-1" y="-1" a="${-3.1415926535 / 4 * 3}"/>
-    <xacro:swerve id="rl" l="${l}" w="${w}" x="-1" y="1" a="${3.1415926535 / 4 * 3}"/>
+    <xacro:swerve id="fl" l="${l}" w="${w}" x="1" y="1" a="${pi / 4}"/>
+    <xacro:swerve id="fr" l="${l}" w="${w}" x="1" y="-1" a="${-pi / 4}"/>
+    <xacro:swerve id="rr" l="${l}" w="${w}" x="-1" y="-1" a="${-pi / 4 * 3}"/>
+    <xacro:swerve id="rl" l="${l}" w="${w}" x="-1" y="1" a="${pi / 4 * 3}"/>
     <xacro:swerve_indicator l="${l}" w="${w}" x="1" y="1"/>
   </xacro:macro>
